Commit message: implement torque_control on one of ur5 arms separately

File: ur5_description/urdf/ur5_right_joint_limited_robot.urdf (robot description, URDF)
Before this commit: robot ur5, 19 links, 18 joints
Links:
- removed link base_l
- removed link base_link_l
- removed link forearm_link_l
- removed link shoulder_link_l
- removed link tool0_l
- removed link upper_arm_link_l
- removed link wrist_1_link_l
- removed link wrist_2_link_l
- removed link wrist_3_link_l
Joints:
- removed joint base_link_l-base_fixed_joint
- removed joint elbow_joint_l
- removed joint shoulder_lift_joint_l
- removed joint shoulder_pan_joint_l
- removed joint world_joint_l
- removed joint wrist_1_joint_l
- removed joint wrist_2_joint_l
- removed joint wrist_3_joint_l
- removed joint wrist_3_link_l-tool0_fixed_joint

Commit message: right ur5 setup created

File: ur5_description/urdf/ur5_right_joint_limited_robot.urdf (robot description, URDF)
Before this commit: robot ur5, 10 links, 9 joints
Links:
- added link ee_link_r; collision box size=0.01 0.01 0.01
- added link obj, mass .5; collision box size=0.05 .2174 0.05; visual box size=0.05 .2174 0.05
Joints:
- added joint ee_fixed_joint_r: type fixed, parent wrist_3_link_r, child ee_link_r, origin xyz=0.0 0.0823 0.0 rpy=0.0 0.0 1.57079632679
- added joint wrist_3_to_obj_joint_r: type fixed, parent wrist_3_link_r, child obj, origin xyz=0 0 0 rpy=0 0 0
