Commit message: add left arm urdf model

File: ur5_description/urdf/ur5_left_joint_limited_robot.urdf (robot description, URDF)
Before this commit: robot ur5, 11 links, 10 joints
Links:
- removed link base
- removed link base_link
- removed link ee_link
- removed link forearm_link
- removed link shoulder_link
- removed link tool0
- removed link upper_arm_link
- removed link wrist_1_link
- removed link wrist_2_link
- removed link wrist_3_link
- added link base_l
- added link base_link_l, mass 4.0; collision mesh filename=package://ur5_description/meshes/ur5/collision/base.stl; visual mesh filename=package://ur5_description/meshes/ur5/visual/base.dae
- added link forearm_link_l, mass 2.275; collision mesh filename=package://ur5_description/meshes/ur5/collision/forearm.stl; visual mesh filename=package://ur5_description/meshes/ur5/visual/forearm.dae
- added link shoulder_link_l, mass 3.7; collision mesh filename=package://ur5_description/meshes/ur5/collision/shoulder.stl; visual mesh filename=package://ur5_description/meshes/ur5/visual/shoulder.dae
- added link tool0_l
- added link upper_arm_link_l, mass 8.393; collision mesh filename=package://ur5_description/meshes/ur5/collision/upperarm.stl; visual mesh filename=package://ur5_description/meshes/ur5/visual/upperarm.dae
- added link wrist_1_link_l, mass 1.219; collision mesh filename=package://ur5_description/meshes/ur5/collision/wrist1.stl; visual mesh filename=package://ur5_description/meshes/ur5/visual/wrist1.dae
- added link wrist_2_link_l, mass 1.219; collision mesh filename=package://ur5_description/meshes/ur5/collision/wrist2.stl; visual mesh filename=package://ur5_description/meshes/ur5/visual/wrist2.dae
- added link wrist_3_link_l, mass 0.1879; collision mesh filename=package://ur5_description/meshes/ur5/collision/wrist3.stl; visual mesh filename=package://ur5_description/meshes/ur5/visual/wrist3.dae
Joints:
- removed joint base_link-base_fixed_joint
- removed joint ee_fixed_joint
- removed joint elbow_joint
- removed joint shoulder_lift_joint
- removed joint shoulder_pan_joint
- removed joint world_joint
- removed joint wrist_1_joint
- removed joint wrist_2_joint
- removed joint wrist_3_joint
- removed joint wrist_3_link-tool0_fixed_joint
- added joint base_link_l-base_fixed_joint: type fixed, parent base_link_l, child base_l, origin xyz=0 0 0 rpy=0 0 -3.14159265359
- added joint elbow_joint_l: type revolute, parent upper_arm_link_l, child forearm_link_l, origin xyz=0.0 -0.1197 0.425 rpy=0.0 -1.5708 0.0, axis 0 1 0, limit lower=-3.14159265359 upper=3.14159265359 effort=150.0 velocity=3.15
- added joint shoulder_lift_joint_l: type revolute, parent shoulder_link_l, child upper_arm_link_l, origin xyz=0.0 0.13585 0.0 rpy=0.0 0.0 0.0, axis 0 1 0, limit lower=-3.14159265359 upper=3.14159265359 effort=150.0 velocity=3.15
- added joint shoulder_pan_joint_l: type revolute, parent base_link_l, child shoulder_link_l, origin xyz=0.0 0.0 0.089159 rpy=0.0 0.0 3.14159265359, axis 0 0 1, limit lower=-3.14159265359 upper=3.14159265359 effort=150.0 velocity=3.15
- added joint world_joint_l: type fixed, parent world, child base_link_l, origin xyz=0.0 0.3 0.0 rpy=0.0 0.0 0.0
- added joint wrist_1_joint_l: type revolute, parent forearm_link_l, child wrist_1_link_l, origin xyz=0.0 0.0 0.39225 rpy=0.0 1.57079632679 0.0, axis 0 1 0, limit lower=-3.14159265359 upper=3.14159265359 effort=28.0 velocity=3.2
- added joint wrist_2_joint_l: type revolute, parent wrist_1_link_l, child wrist_2_link_l, origin xyz=0.0 0.093 0.0 rpy=0.0 0.0 0.0, axis 0 0 1, limit lower=-3.14159265359 upper=3.14159265359 effort=28.0 velocity=3.2
- added joint wrist_3_joint_l: type revolute, parent wrist_2_link_l, child wrist_3_link_l, origin xyz=0.0 0.0 0.09465 rpy=0.0 0.0 0.0, axis 0 1 0, limit lower=-3.14159265359 upper=3.14159265359 effort=28.0 velocity=3.2
- added joint wrist_3_link_l-tool0_fixed_joint: type fixed, parent wrist_3_link_l, child tool0_l, origin xyz=0 0.0823 0 rpy=-1.57079632679 0 0

Commit message: left ur5 setup created

File: ur5_description/urdf/ur5_left_joint_limited_robot.urdf (robot description, URDF)
Before this commit: robot ur5, 10 links, 9 joints
Links:
- added link ee_link_l; collision box size=0.01 0.01 0.01
Joints:
- added joint ee_fixed_joint_l: type fixed, parent wrist_3_link_l, child ee_link_l, origin xyz=0.0 0.0823 0.0 rpy=0.0 0.0 1.57079632679
