Commit message: two arms control separately :)

File: ur5_description/urdf/ur5.urdf.xacro (robot description, xacro)
@@ -354,4 +354,5 @@
       <child link = "${prefix}shoulder_link_l" />
       <origin xyz="0.0 0.0 ${shoulder_height}" rpy="0.0 0.0 ${pi}" />
+      <!-- <origin xyz="0.0 0.0 ${shoulder_height}" rpy="0.0 0.0 0.0" /> -->
       <axis xyz="0 0 1" />
       <xacro:unless value="${joint_limited}">
@@ -416,4 +417,5 @@
       <child link = "${prefix}forearm_link_l" />
       <origin xyz="0.0 ${elbow_offset} ${upper_arm_length}" rpy="0.0 ${-pi / 2.0} 0.0" />
+      <!-- <origin xyz="0.0 ${elbow_offset} ${upper_arm_length}" rpy="0.0 0.0 0.0" /> -->
       <axis xyz="0 1 0" />
       <xacro:unless value="${joint_limited}">
@@ -447,4 +449,5 @@
       <child link = "${prefix}wrist_1_link_l" />
       <origin xyz="0.0 0.0 ${forearm_length}" rpy="0.0 ${pi / 2.0} 0.0" />
+      <!-- <origin xyz="0.0 0.0 ${forearm_length}" rpy="0.0 0.0 0.0" /> -->
       <axis xyz="0 1 0" />
       <xacro:unless value="${joint_limited}">

File: ur5_description/urdf/ur5_left_joint_limited_robot.urdf (robot description, URDF)
Before this commit: robot ur5, 10 links, 9 joints
Links:
- added link ee_link_l; collision box size=0.01 0.01 0.01
Joints:
- added joint ee_fixed_joint_l: type fixed, parent wrist_3_link_l, child ee_link_l, origin xyz=0.0 0.0823 0.0 rpy=0.0 0.0 1.57079632679
- joint shoulder_pan_joint_l: origin xyz=0.0 0.0 0.089159 rpy=0.0 0.0 3.14159265359 -> xyz=0.0 0.0 0.089159 rpy=0.0 0.0 3.141592

File: ur5_description/urdf/ur5_right_joint_limited_robot.urdf (robot description, URDF)
Before this commit: robot ur5, 10 links, 9 joints
Links:
- added link ee_link_r; collision box size=0.01 0.01 0.01
Joints:
- added joint ee_fixed_joint_r: type fixed, parent wrist_3_link_r, child ee_link_r, origin xyz=0.0 0.0823 0.0 rpy=0.0 0.0 1.57079632679

Commit message: add obj anf fix to both wrists

File: ur5_description/urdf/ur5.urdf.xacro (robot description, xacro)
@@ -46,5 +46,5 @@
   <xacro:property name="wrist_2_length" value="${ur5_d5}" />
   <xacro:property name="wrist_3_length" value="${ur5_d6}" />
-  <xacro:property name="obj_length" value="0.2" />
+  <xacro:property name="obj_length" value="0.2174" />
   <!--property name="shoulder_height" value="0.089159" /-->
   <!--property name="shoulder_offset" value="0.13585" /-->  <!-- shoulder_offset - elbow_offset + wrist_1_length = 0.10915 -->
@@ -274,5 +274,271 @@
       </xacro:cylinder_inertial>
     </link>
-    <!-- <joint name="box_R_fixed" type="fixed">
+    <joint name="${prefix}ee_fixed_joint_r" type="fixed">
+      <parent link="${prefix}wrist_3_link_r" />
+      <child link = "${prefix}ee_link_r" />
+      <origin xyz="0.0 ${wrist_3_length} 0.0" rpy="0.0 0.0 ${pi/2.0}" />
+    </joint>
+    <link name="${prefix}ee_link_r">
+      <collision>
+        <geometry>
+          <box size="0.01 0.01 0.01"/>
+        </geometry>
+        <origin rpy="0 0 0" xyz="-0.01 0 0"/>
+      </collision>
+    </link>
+    <xacro:ur_arm_transmission prefix="${prefix}" />
+    <xacro:ur_arm_gazebo prefix="${prefix}" />
+    <!-- ROS base_link to UR 'Base' Coordinates transform -->
+    <link name="${prefix}base_r"/>
+    <joint name="${prefix}base_link_r-base_fixed_joint" type="fixed">
+      <!-- NOTE: this rotation is only needed as long as base_link itself is
+                 not corrected wrt the real robot (ie: rotated over 180
+                 degrees)
+      -->
+      <origin xyz="0 0 0" rpy="0 0 ${-pi}"/>
+      <parent link="${prefix}base_link_r"/>
+      <child link="${prefix}base_r"/>
+    </joint>
+    <!-- Frame coincident with all-zeros TCP on UR controller -->
+    <link name="${prefix}tool0_r"/>
+    <joint name="${prefix}wrist_3_link_r-tool0_fixed_joint" type="fixed">
+      <origin xyz="0 ${wrist_3_length} 0" rpy="${pi/-2.0} 0 0"/>
+      <parent link="${prefix}wrist_3_link_r"/>
+      <child link="${prefix}tool0_r"/>
+    </joint>
+    <link name="${prefix}base_link_l" >
+      <visual>
+        <geometry>
+          <mesh filename="package://ur5_description/meshes/ur5/visual/base.dae" />
+        </geometry>
+        <material name="LightGrey">
+          <color rgba="0.7 0.7 0.7 1.0"/>
+        </material>
+      </visual>
+      <collision>
+        <geometry>
+          <mesh filename="package://ur5_description/meshes/ur5/collision/base.stl" />
+        </geometry>
+      </collision>
+      <xacro:cylinder_inertial radius="0.06" length="0.05" mass="${base_mass}">
+        <origin xyz="0.0 0.0 0.0" rpy="0 0 0" />
+      </xacro:cylinder_inertial>
+    </link>
+    <joint name="${prefix}shoulder_pan_joint_l" type="revolute">
+      <parent link="${prefix}base_link_l" />
+      <child link = "${prefix}shoulder_link_l" />
+      <origin xyz="0.0 0.0 ${shoulder_height}" rpy="0.0 0.0 ${pi}" />
+      <axis xyz="0 0 1" />
+      <xacro:unless value="${joint_limited}">
+        <limit lower="${-2.0 * pi}" upper="${2.0 * pi}" effort="150.0" velocity="3.15"/>
+      </xacro:unless>
+      <xacro:if value="${joint_limited}">
+        <limit lower="${-pi}" upper="${pi}" effort="150.0" velocity="3.15"/>
+      </xacro:if>
+      <dynamics damping="0.0" friction="0.0"/>
+    </joint>
+    <link name="${prefix}shoulder_link_l">
+      <visual>
+        <geometry>
+          <mesh filename="package://ur5_description/meshes/ur5/visual/shoulder.dae" />
+        </geometry>
+        <material name="LightGrey">
+          <color rgba="0.7 0.7 0.7 1.0"/>
+        </material>
+      </visual>
+      <collision>
+        <geometry>
+          <mesh filename="package://ur5_description/meshes/ur5/collision/shoulder.stl" />
+        </geometry>
+      </collision>
+      <xacro:cylinder_inertial radius="0.06" length="0.15" mass="${shoulder_mass}">
+        <origin xyz="0.0 0.0 0.0" rpy="0 0 0" />
+      </xacro:cylinder_inertial>
+    </link>
+    <joint name="${prefix}shoulder_lift_joint_l" type="revolute">
+      <parent link="${prefix}shoulder_link_l" />
+      <child link = "${prefix}upper_arm_link_l" />
+      <origin xyz="0.0 ${shoulder_offset} 0.0" rpy="0.0 0.0 0.0" />
+      <axis xyz="0 1 0" />
+      <xacro:unless value="${joint_limited}">
+        <limit lower="${-2.0 * pi}" upper="${2.0 * pi}" effort="150.0" velocity="3.15"/>
+      </xacro:unless>
+      <xacro:if value="${joint_limited}">
+        <limit lower="${-pi}" upper="${pi}" effort="150.0" velocity="3.15"/>
+      </xacro:if>
+      <dynamics damping="0.0" friction="0.0"/>
+    </joint>
+    <link name="${prefix}upper_arm_link_l">
+      <visual>
+        <geometry>
+          <mesh filename="package://ur5_description/meshes/ur5/visual/upperarm.dae" />
+        </geometry>
+        <material name="LightGrey">
+          <color rgba="0.7 0.7 0.7 1.0"/>
+        </material>
+      </visual>
+      <collision>
+        <geometry>
+          <mesh filename="package://ur5_description/meshes/ur5/collision/upperarm.stl" />
+        </geometry>
+      </collision>
+      <xacro:cylinder_inertial radius="0.06" length="0.56" mass="${upper_arm_mass}">
+        <origin xyz="0.0 0.0 0.28" rpy="0 0 0" />
+      </xacro:cylinder_inertial>
+    </link>
+    <joint name="${prefix}elbow_joint_l" type="revolute">
+      <parent link="${prefix}upper_arm_link_l" />
+      <child link = "${prefix}forearm_link_l" />
+      <origin xyz="0.0 ${elbow_offset} ${upper_arm_length}" rpy="0.0 ${-pi / 2.0} 0.0" />
+      <axis xyz="0 1 0" />
+      <xacro:unless value="${joint_limited}">
+        <limit lower="${-pi}" upper="${pi}" effort="150.0" velocity="3.15"/>
+      </xacro:unless>
+      <xacro:if value="${joint_limited}">
+        <limit lower="${-pi}" upper="${pi}" effort="150.0" velocity="3.15"/>
+      </xacro:if>
+      <dynamics damping="0.0" friction="0.0"/>
+    </joint>
+    <link name="${prefix}forearm_link_l">
+      <visual>
+        <geometry>
+          <mesh filename="package://ur5_description/meshes/ur5/visual/forearm.dae" />
+        </geometry>
+        <material name="LightGrey">
+          <color rgba="0.7 0.7 0.7 1.0"/>
+        </material>
+      </visual>
+      <collision>
+        <geometry>
+          <mesh filename="package://ur5_description/meshes/ur5/collision/forearm.stl" />
+        </geometry>
+      </collision>
+      <xacro:cylinder_inertial radius="0.06" length="0.5" mass="${forearm_mass}">
+        <origin xyz="0.0 0.0 0.25" rpy="0 0 0" />
+      </xacro:cylinder_inertial>
+    </link>
+    <joint name="${prefix}wrist_1_joint_l" type="revolute">
+      <parent link="${prefix}forearm_link_l" />
+      <child link = "${prefix}wrist_1_link_l" />
+      <origin xyz="0.0 0.0 ${forearm_length}" rpy="0.0 ${pi / 2.0} 0.0" />
+      <axis xyz="0 1 0" />
+      <xacro:unless value="${joint_limited}">
+        <limit lower="${-2.0 * pi}" upper="${2.0 * pi}" effort="28.0" velocity="3.2"/>
+      </xacro:unless>
+      <xacro:if value="${joint_limited}">
+        <limit lower="${-pi}" upper="${pi}" effort="28.0" velocity="3.2"/>
+      </xacro:if>
+      <dynamics damping="0.0" friction="0.0"/>
+    </joint>
+    <link name="${prefix}wrist_1_link_l">
+      <visual>
+        <geometry>
+          <mesh filename="package://ur5_description/meshes/ur5/visual/wrist1.dae" />
+        </geometry>
+        <material name="LightGrey">
+          <color rgba="0.7 0.7 0.7 1.0"/>
+        </material>
+      </visual>
+      <collision>
+        <geometry>
+          <mesh filename="package://ur5_description/meshes/ur5/collision/wrist1.stl" />
+        </geometry>
+      </collision>
+      <xacro:cylinder_inertial radius="0.6" length="0.12" mass="${wrist_1_mass}">
+        <origin xyz="0.0 0.0 0.0" rpy="0 0 0" />
+      </xacro:cylinder_inertial>
+    </link>
+    <joint name="${prefix}wrist_2_joint_l" type="revolute">
+      <parent link="${prefix}wrist_1_link_l" />
+      <child link = "${prefix}wrist_2_link_l" />
+      <origin xyz="0.0 ${wrist_1_length} 0.0" rpy="0.0 0.0 0.0" />
+      <axis xyz="0 0 1" />
+      <xacro:unless value="${joint_limited}">
+        <limit lower="${-2.0 * pi}" upper="${2.0 * pi}" effort="28.0" velocity="3.2"/>
+      </xacro:unless>
+      <xacro:if value="${joint_limited}">
+        <limit lower="${-pi}" upper="${pi}" effort="28.0" velocity="3.2"/>
+      </xacro:if>
+      <dynamics damping="0.0" friction="0.0"/>
+    </joint>
+    <link name="${prefix}wrist_2_link_l">
+      <visual>
+        <geometry>
+          <mesh filename="package://ur5_description/meshes/ur5/visual/wrist2.dae" />
+        </geometry>
+        <material name="LightGrey">
+          <color rgba="0.7 0.7 0.7 1.0"/>
+        </material>
+      </visual>
+      <collision>
+        <geometry>
+          <mesh filename="package://ur5_description/meshes/ur5/collision/wrist2.stl" />
+        </geometry>
+      </collision>
+      <xacro:cylinder_inertial radius="0.6" length="0.12" mass="${wrist_2_mass}">
+        <origin xyz="0.0 0.0 0.0" rpy="0 0 0" />
+      </xacro:cylinder_inertial>
+    </link>
+    <joint name="${prefix}wrist_3_joint_l" type="revolute">
+      <parent link="${prefix}wrist_2_link_l" />
+      <child link = "${prefix}wrist_3_link_l" />
+      <origin xyz="0.0 0.0 ${wrist_2_length}" rpy="0.0 0.0 0.0" />
+      <axis xyz="0 1 0" />
+      <xacro:unless value="${joint_limited}">
+        <limit lower="${-2.0 * pi}" upper="${2.0 * pi}" effort="28.0" velocity="3.2"/>
+      </xacro:unless>
+      <xacro:if value="${joint_limited}">
+        <limit lower="${-pi}" upper="${pi}" effort="28.0" velocity="3.2"/>
+      </xacro:if>
+      <dynamics damping="0.0" friction="0.0"/>
+    </joint>
+    <link name="${prefix}wrist_3_link_l">
+      <visual>
+        <geometry>
+          <mesh filename="package://ur5_description/meshes/ur5/visual/wrist3.dae" />
+        </geometry>
+        <material name="LightGrey">
+          <color rgba="0.7 0.7 0.7 1.0"/>
+        </material>
+      </visual>
+      <collision>
+        <geometry>
+          <mesh filename="package://ur5_description/meshes/ur5/collision/wrist3.stl" />
+        </geometry>
+      </collision>
+      <xacro:cylinder_inertial radius="0.6" length="0.12" mass="${wrist_3_mass}">
+        <origin xyz="0.0 0.0 0.0" rpy="0 0 0" />
+      </xacro:cylinder_inertial>
+    </link>
+    <joint name="${prefix}ee_fixed_joint_l" type="fixed">
+      <parent link="${prefix}wrist_3_link_l" />
+      <child link = "${prefix}ee_link_l" />
+      <origin xyz="0.0 ${wrist_3_length} 0.0" rpy="0.0 0.0 ${pi/2.0}" />
+    </joint>
+    <link name="${prefix}ee_link_l">
+      <collision>
+        <geometry>
+          <box size="0.01 0.01 0.01"/>
+        </geometry>
+        <origin rpy="0 0 0" xyz="-0.01 0 0"/>
+      </collision>
+    </link>
+    <xacro:ur_arm_transmission prefix="${prefix}" />
+    <xacro:ur_arm_gazebo prefix="${prefix}" />
+    <!-- ROS base_link to UR 'Base' Coordinates transform -->
+    <link name="${prefix}base_l"/>
+    <joint name="${prefix}base_link_l-base_fixed_joint" type="fixed">
+      <origin xyz="0 0 0" rpy="0 0 ${-pi}"/>
+      <parent link="${prefix}base_link_l"/>
+      <child link="${prefix}base_l"/>
+    </joint>
+    <!-- Frame coincident with all-zeros TCP on UR controller -->
+    <link name="${prefix}tool0_l"/>
+    <joint name="${prefix}wrist_3_link_l-tool0_fixed_joint" type="fixed">
+      <origin xyz="0 ${wrist_3_length} 0" rpy="${pi/-2.0} 0 0"/>
+      <parent link="${prefix}wrist_3_link_l"/>
+      <child link="${prefix}tool0_l"/>
+    </joint>
+    <joint name="wrist_3_to_obj_joint_r" type="fixed">
         <origin rpy="0 0 0" xyz="0 0 0"/>
         <parent link="${prefix}wrist_3_link_r"/>
@@ -285,5 +551,5 @@
                 <box size="0.05 ${obj_length} 0.05"/>
             </geometry>
-            <material name="green"/>
+            <material name="LightGreen"/>
         </visual>
         <collision>
@@ -298,274 +564,22 @@
             <inertia ixx="1" ixy="0" ixz="0" iyy="1" iyz="0" izz="1"/>
         </inertial>
-    </link> -->
-    <joint name="${prefix}ee_fixed_joint_r" type="fixed">
-      <parent link="${prefix}wrist_3_link_r" />
-      <child link = "${prefix}ee_link_r" />
-      <origin xyz="0.0 ${wrist_3_length} 0.0" rpy="0.0 0.0 ${pi/2.0}" />
-    </joint>
-    <link name="${prefix}ee_link_r">
-      <collision>
-        <geometry>
-          <box size="0.01 0.01 0.01"/>
-        </geometry>
-        <origin rpy="0 0 0" xyz="-0.01 0 0"/>
-      </collision>
-    </link>
-    <xacro:ur_arm_transmission prefix="${prefix}" />
-    <xacro:ur_arm_gazebo prefix="${prefix}" />
-    <!-- ROS base_link to UR 'Base' Coordinates transform -->
-    <link name="${prefix}base_r"/>
-    <joint name="${prefix}base_link_r-base_fixed_joint" type="fixed">
-      <!-- NOTE: this rotation is only needed as long as base_link itself is
-                 not corrected wrt the real robot (ie: rotated over 180
-                 degrees)
-      -->
-      <origin xyz="0 0 0" rpy="0 0 ${-pi}"/>
-      <parent link="${prefix}base_link_r"/>
-      <child link="${prefix}base_r"/>
-    </joint>
-    <!-- Frame coincident with all-zeros TCP on UR controller -->
-    <link name="${prefix}tool0_r"/>
-    <joint name="${prefix}wrist_3_link_r-tool0_fixed_joint" type="fixed">
-      <origin xyz="0 ${wrist_3_length} 0" rpy="${pi/-2.0} 0 0"/>
-      <parent link="${prefix}wrist_3_link_r"/>
-      <child link="${prefix}tool0_r"/>
-    </joint>
-    <link name="${prefix}base_link_l" >
-      <visual>
-        <geometry>
-          <mesh filename="package://ur5_description/meshes/ur5/visual/base.dae" />
-        </geometry>
-        <material name="LightGrey">
-          <color rgba="0.7 0.7 0.7 1.0"/>
-        </material>
-      </visual>
-      <collision>
-        <geometry>
-          <mesh filename="package://ur5_description/meshes/ur5/collision/base.stl" />
-        </geometry>
-      </collision>
-      <xacro:cylinder_inertial radius="0.06" length="0.05" mass="${base_mass}">
-        <origin xyz="0.0 0.0 0.0" rpy="0 0 0" />
-      </xacro:cylinder_inertial>
-    </link>
-    <joint name="${prefix}shoulder_pan_joint_l" type="revolute">
-      <parent link="${prefix}base_link_l" />
-      <child link = "${prefix}shoulder_link_l" />
-      <origin xyz="0.0 0.0 ${shoulder_height}" rpy="0.0 0.0 ${pi}" />
-      <!-- <origin xyz="0.0 0.0 ${shoulder_height}" rpy="0.0 0.0 0.0" /> -->
-      <axis xyz="0 0 1" />
-      <xacro:unless value="${joint_limited}">
-        <limit lower="${-2.0 * pi}" upper="${2.0 * pi}" effort="150.0" velocity="3.15"/>
-      </xacro:unless>
-      <xacro:if value="${joint_limited}">
-        <limit lower="${-pi}" upper="${pi}" effort="150.0" velocity="3.15"/>
-      </xacro:if>
-      <dynamics damping="0.0" friction="0.0"/>
-    </joint>
-    <link name="${prefix}shoulder_link_l">
-      <visual>
-        <geometry>
-          <mesh filename="package://ur5_description/meshes/ur5/visual/shoulder.dae" />
-        </geometry>
-        <material name="LightGrey">
-          <color rgba="0.7 0.7 0.7 1.0"/>
-        </material>
-      </visual>
-      <collision>
-        <geometry>
-          <mesh filename="package://ur5_description/meshes/ur5/collision/shoulder.stl" />
-        </geometry>
-      </collision>
-      <xacro:cylinder_inertial radius="0.06" length="0.15" mass="${shoulder_mass}">
-        <origin xyz="0.0 0.0 0.0" rpy="0 0 0" />
-      </xacro:cylinder_inertial>
-    </link>
-    <joint name="${prefix}shoulder_lift_joint_l" type="revolute">
-      <parent link="${prefix}shoulder_link_l" />
-      <child link = "${prefix}upper_arm_link_l" />
-      <origin xyz="0.0 ${shoulder_offset} 0.0" rpy="0.0 0.0 0.0" />
-      <axis xyz="0 1 0" />
-      <xacro:unless value="${joint_limited}">
-        <limit lower="${-2.0 * pi}" upper="${2.0 * pi}" effort="150.0" velocity="3.15"/>
-      </xacro:unless>
-      <xacro:if value="${joint_limited}">
-        <limit lower="${-pi}" upper="${pi}" effort="150.0" velocity="3.15"/>
-      </xacro:if>
-      <dynamics damping="0.0" friction="0.0"/>
-    </joint>
-    <link name="${prefix}upper_arm_link_l">
-      <visual>
-        <geometry>
-          <mesh filename="package://ur5_description/meshes/ur5/visual/upperarm.dae" />
-        </geometry>
-        <material name="LightGrey">
-          <color rgba="0.7 0.7 0.7 1.0"/>
-        </material>
-      </visual>
-      <collision>
-        <geometry>
-          <mesh filename="package://ur5_description/meshes/ur5/collision/upperarm.stl" />
-        </geometry>
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
Commit message: both arm track circular trajectory alongside each other.

File: ur5_description/urdf/ur5.urdf.xacro (robot description, xacro)
@@ -274,5 +274,5 @@
       </xacro:cylinder_inertial>
     </link>
-    <joint name="${prefix}ee_fixed_joint_r" type="fixed">
+    <!-- <joint name="${prefix}ee_fixed_joint_r" type="fixed">
       <parent link="${prefix}wrist_3_link_r" />
       <child link = "${prefix}ee_link_r" />
@@ -286,5 +286,5 @@
         <origin rpy="0 0 0" xyz="-0.01 0 0"/>
       </collision>
-    </link>
+    </link> -->
     <xacro:ur_arm_transmission prefix="${prefix}" />
     <xacro:ur_arm_gazebo prefix="${prefix}" />
@@ -511,5 +511,5 @@
       </xacro:cylinder_inertial>
     </link>
-    <joint name="${prefix}ee_fixed_joint_l" type="fixed">
+    <!-- <joint name="${prefix}ee_fixed_joint_l" type="fixed">
       <parent link="${prefix}wrist_3_link_l" />
       <child link = "${prefix}ee_link_l" />
@@ -523,5 +523,5 @@
         <origin rpy="0 0 0" xyz="-0.01 0 0"/>
       </collision>
-    </link>
+    </link> -->
     <xacro:ur_arm_transmission prefix="${prefix}" />
     <xacro:ur_arm_gazebo prefix="${prefix}" />
@@ -540,5 +540,5 @@
       <child link="${prefix}tool0_l"/>
     </joint>
-    <joint name="wrist_3_to_obj_joint_r" type="fixed">
+    <!-- <joint name="wrist_3_to_obj_joint_r" type="fixed">
         <origin rpy="0 0 0" xyz="0 0 0"/>
         <parent link="${prefix}wrist_3_link_r"/>
@@ -581,5 +581,5 @@
             </physics>
         </joint>
-    </gazebo>
+    </gazebo> -->
   </xacro:macro>
 </robot>

File: ur5_description/urdf/ur5_left_joint_limited_robot.urdf (robot description, URDF)
Before this commit: robot ur5, 11 links, 10 joints
Links:
- removed link ee_link_l
Joints:
- removed joint ee_fixed_joint_l

File: ur5_description/urdf/ur5_right_joint_limited_robot.urdf (robot description, URDF)
Before this commit: robot ur5, 11 links, 10 joints
Links:
- removed link ee_link_r
Joints:
- removed joint ee_fixed_joint_r

Commit message: two arms, no object, follow same orientation separately.

File: ur5_description/urdf/ur5.urdf.xacro (robot description, xacro)
@@ -274,5 +274,5 @@
       </xacro:cylinder_inertial>
     </link>
-    <!-- <joint name="${prefix}ee_fixed_joint_r" type="fixed">
+    <joint name="${prefix}ee_fixed_joint_r" type="fixed">
       <parent link="${prefix}wrist_3_link_r" />
       <child link = "${prefix}ee_link_r" />
@@ -286,5 +286,5 @@
         <origin rpy="0 0 0" xyz="-0.01 0 0"/>
       </collision>
-    </link> -->
+    </link>
     <xacro:ur_arm_transmission prefix="${prefix}" />
     <xacro:ur_arm_gazebo prefix="${prefix}" />
@@ -511,5 +511,5 @@
       </xacro:cylinder_inertial>
     </link>
-    <!-- <joint name="${prefix}ee_fixed_joint_l" type="fixed">
+    <joint name="${prefix}ee_fixed_joint_l" type="fixed">
       <parent link="${prefix}wrist_3_link_l" />
       <child link = "${prefix}ee_link_l" />
@@ -523,5 +523,5 @@
         <origin rpy="0 0 0" xyz="-0.01 0 0"/>
       </collision>
-    </link> -->
+    </link>
     <!-- ROS base_link to UR 'Base' Coordinates transform -->
     <link name="${prefix}base_l"/>

File: ur5_description/urdf/ur5_right_joint_limited_robot.urdf (robot description, URDF)
Before this commit: robot ur5, 12 links, 11 joints
Links:
- removed link obj
Joints:
- removed joint wrist_3_to_obj_joint_r

Commit message: seems linear control is implemented.

File: ur5_description/urdf/ur5.urdf.xacro (robot description, xacro)
@@ -538,5 +538,5 @@
       <child link="${prefix}tool0_l"/>
     </joint>
-    <!-- <joint name="wrist_3_to_obj_joint_r" type="fixed">
+    <joint name="wrist_3_to_obj_joint_r" type="fixed">
         <origin rpy="0 0 0" xyz="0 0 0"/>
         <parent link="${prefix}wrist_3_link_r"/>
@@ -567,5 +567,5 @@
             <parent>wrist_3_link_l</parent>
             <child>obj</child>
-            <pose>-0.02 0 0 0 0 0</pose>
+            <pose>0 ${obj_length + wrist_3_length} 0 0 0 0</pose>
             <physics>
                 <ode>
@@ -579,5 +579,5 @@
             </physics>
         </joint>
-    </gazebo> -->
+    </gazebo>
   </xacro:macro>
 </robot>

File: ur5_description/urdf/ur5_right_joint_limited_robot.urdf (robot description, URDF)
Before this commit: robot ur5, 11 links, 10 joints
Links:
- added link obj, mass .5; collision box size=0.05 .2174 0.05; visual box size=0.05 .2174 0.05
Joints:
- added joint wrist_3_to_obj_joint_r: type fixed, parent wrist_3_link_r, child obj, origin xyz=0 0 0 rpy=0 0 0
