Commit message: fix linear and angular trajectory tracking for bi-manual ur5

File: ur5_description/urdf/ur5.urdf.xacro (robot description, xacro)
@@ -122,5 +122,6 @@
       <parent link="${prefix}shoulder_link_r" />
       <child link = "${prefix}upper_arm_link_r" />
-      <origin xyz="0.0 ${shoulder_offset} 0.0" rpy="0.0 0.0 0.0" />
+      <!-- <origin xyz="0.0 ${shoulder_offset} 0.0" rpy="0.0 0.0 0.0" /> -->
+      <origin xyz="0.0 ${shoulder_offset} 0.0" rpy="0.0 ${pi / 6.0} 0.0" />
       <axis xyz="0 1 0" />
       <xacro:unless value="${joint_limited}">
@@ -153,4 +154,5 @@
       <parent link="${prefix}upper_arm_link_r" />
       <child link = "${prefix}forearm_link_r" />
+      <!-- <origin xyz="0.0 ${elbow_offset} ${upper_arm_length}" rpy="0.0 ${pi / 2.0} 0.0" /> -->
       <origin xyz="0.0 ${elbow_offset} ${upper_arm_length}" rpy="0.0 ${pi / 2.0} 0.0" />
       <axis xyz="0 1 0" />
@@ -184,5 +186,6 @@
       <parent link="${prefix}forearm_link_r" />
       <child link = "${prefix}wrist_1_link_r" />
-      <origin xyz="0.0 0.0 ${forearm_length}" rpy="0.0 ${-pi / 2.0} 0.0" />
+      <!-- <origin xyz="0.0 0.0 ${forearm_length}" rpy="0.0 ${-pi / 2.0} 0.0" /> -->
+      <origin xyz="0.0 0.0 ${forearm_length}" rpy="0.0 ${pi / 3.0} 0.0" />
       <axis xyz="0 1 0" />
       <xacro:unless value="${joint_limited}">
@@ -359,5 +362,6 @@
       <parent link="${prefix}shoulder_link_l" />
       <child link = "${prefix}upper_arm_link_l" />
-      <origin xyz="0.0 ${shoulder_offset} 0.0" rpy="0.0 0.0 0.0" />
+      <!-- <origin xyz="0.0 ${shoulder_offset} 0.0" rpy="0.0 0.0 0.0" /> -->
+      <origin xyz="0.0 ${shoulder_offset} 0.0" rpy="0.0 ${-pi / 6.0} 0.0" />
       <axis xyz="0 1 0" />
       <xacro:unless value="${joint_limited}">
@@ -421,5 +425,6 @@
       <parent link="${prefix}forearm_link_l" />
       <child link = "${prefix}wrist_1_link_l" />
-      <origin xyz="0.0 0.0 ${forearm_length}" rpy="0.0 ${pi / 2.0} 0.0" />
+      <!-- <origin xyz="0.0 0.0 ${forearm_length}" rpy="0.0 ${pi / 2.0} 0.0" /> -->
+      <origin xyz="0.0 0.0 ${forearm_length}" rpy="0.0 ${-pi / 3.0} 0.0" />
       <axis xyz="0 1 0" />
       <xacro:unless value="${joint_limited}">
@@ -539,5 +544,5 @@
     </joint>
     <joint name="wrist_3_to_obj_joint_r" type="fixed">
-        <origin rpy="0 0 0" xyz="0 0 0"/>
+        <origin rpy="0 0 0" xyz="0 ${wrist_3_length} 0"/>
         <parent link="${prefix}wrist_3_link_r"/>
         <child link="obj"/>
@@ -545,5 +550,5 @@
     <link name="obj">
         <visual>
-            <origin rpy="0 0 0" xyz="0.0 ${obj_length/2 + wrist_3_length} 0.0"/>
+            <origin rpy="0 0 0" xyz="0.0 ${obj_length/2} 0.0"/>
             <geometry>
                 <box size="0.05 ${obj_length} 0.05"/>
@@ -552,5 +557,5 @@
         </visual>
         <collision>
-            <origin rpy="0 0 0" xyz="0.0 ${obj_length/2 + wrist_3_length} 0.0"/>
+            <origin rpy="0 0 0" xyz="0.0 ${obj_length/2} 0.0"/>
             <geometry>
                 <box size="0.05 ${obj_length} 0.05"/>
@@ -558,7 +563,7 @@
         </collision>
         <inertial>
-            <origin rpy="0 0 0" xyz="0.0 ${obj_length/2 + wrist_3_length} 0.0"/>
+            <origin rpy="0 0 0" xyz="0.0 ${obj_length/2} 0.0"/>
             <mass value="${obj_mass}"/>
-            <inertia ixx="1" ixy="0" ixz="0" iyy="1" iyz="0" izz="1"/>
+            <inertia ixx=".0021" ixy="0" ixz="0" iyy=".00021" iyz="0" izz=".0021"/>
         </inertial>
     </link>

File: ur5_description/urdf/ur5_left_joint_limited_robot.urdf (robot description, URDF)
Before this commit: robot ur5, 11 links, 10 joints
Joints:
- joint shoulder_lift_joint_l: origin xyz=0.0 0.13585 0.0 rpy=0.0 0.0 0.0 -> xyz=0.0 0.13585 0.0 rpy=0.0 -.5236 0.0
- joint wrist_1_joint_l: origin xyz=0.0 0.0 0.39225 rpy=0.0 1.57079632679 0.0 -> xyz=0.0 0.0 0.39225 rpy=0.0 -1.047 0.0

File: ur5_description/urdf/ur5_right_joint_limited_robot.urdf (robot description, URDF)
Before this commit: robot ur5, 12 links, 11 joints
Links:
- removed link obj
Joints:
- removed joint wrist_3_to_obj_joint_r
- joint shoulder_lift_joint_r: origin xyz=0.0 0.13585 0.0 rpy=0.0 0.0 0.0 -> xyz=0.0 0.13585 0.0 rpy=0.0 .5236 0.0
- joint wrist_1_joint_r: origin xyz=0.0 0.0 0.39225 rpy=0.0 -1.57079632679 0.0 -> xyz=0.0 0.0 0.39225 rpy=0.0 1.047 0.0

Commit message: modify ur5 urdf model: change COM positions, values, and inertias

File: ur5_description/urdf/ur5.urdf.xacro (robot description, xacro)
@@ -11,5 +11,5 @@
   <xacro:property name="wrist_2_mass" value="1.2190" />
   <xacro:property name="wrist_3_mass" value="0.1879" />
-  <xacro:property name="obj_mass" value="0.5" />
+  <xacro:property name="obj_mass" value="1" />
   <xacro:property name="shoulder_cog" value="0.0 0.00193 -0.02561" />
   <xacro:property name="upper_arm_cog" value="0.0 -0.024201 0.2125" />
@@ -47,12 +47,4 @@
   <xacro:property name="wrist_3_length" value="${ur5_d6}" />
   <xacro:property name="obj_length" value="0.2174" />
-  <!--property name="shoulder_height" value="0.089159" /-->
-  <!--property name="shoulder_offset" value="0.13585" /-->  <!-- shoulder_offset - elbow_offset + wrist_1_length = 0.10915 -->
-  <!--property name="upper_arm_length" value="0.42500" /-->
-  <!--property name="elbow_offset" value="0.1197" /-->       <!-- CAD measured -->
-  <!--property name="forearm_length" value="0.39225" /-->
-  <!--property name="wrist_1_length" value="0.093" /-->     <!-- CAD measured -->
-  <!--property name="wrist_2_length" value="0.09465" /-->   <!-- In CAD this distance is 0.930, but in the spec it is 0.09465 -->
-  <!--property name="wrist_3_length" value="0.0823" /-->
   <xacro:property name="shoulder_radius" value="0.060" />   <!-- manually measured -->
   <xacro:property name="upper_arm_radius" value="0.054" />  <!-- manually measured -->
@@ -122,5 +114,5 @@
       <parent link="${prefix}shoulder_link_r" />
       <child link = "${prefix}upper_arm_link_r" />
-      <!-- <origin xyz="0.0 ${shoulder_offset} 0.0" rpy="0.0 0.0 0.0" /> -->
+      <!-- <origin xyz="0.0 ${shoulder_offset} 0.0" rpy="0.0 ${pi / 2.0} 0.0" /> -->
       <origin xyz="0.0 ${shoulder_offset} 0.0" rpy="0.0 ${pi / 6.0} 0.0" />
       <axis xyz="0 1 0" />
@@ -154,5 +146,5 @@
       <parent link="${prefix}upper_arm_link_r" />
       <child link = "${prefix}forearm_link_r" />
-      <!-- <origin xyz="0.0 ${elbow_offset} ${upper_arm_length}" rpy="0.0 ${pi / 2.0} 0.0" /> -->
+      <!-- <origin xyz="0.0 ${elbow_offset} ${upper_arm_length}" rpy="0.0 0.0 0.0" /> -->
       <origin xyz="0.0 ${elbow_offset} ${upper_arm_length}" rpy="0.0 ${pi / 2.0} 0.0" />
       <axis xyz="0 1 0" />
@@ -179,6 +171,6 @@
         </geometry>
       </collision>
-      <xacro:cylinder_inertial radius="0.06" length="0.5" mass="${forearm_mass}">
-        <origin xyz="0.0 0.0 0.25" rpy="0 0 0" />
+      <xacro:cylinder_inertial radius="0.06" length="${-ur5_a3}" mass="${forearm_mass}">
+        <origin xyz="0.0 0.0 ${-ur5_a3/2.0}" rpy="0 0 0" />
       </xacro:cylinder_inertial>
     </link>
@@ -186,5 +178,6 @@
       <parent link="${prefix}forearm_link_r" />
       <child link = "${prefix}wrist_1_link_r" />
-      <!-- <origin xyz="0.0 0.0 ${forearm_length}" rpy="0.0 ${-pi / 2.0} 0.0" /> -->
+      <!-- <origin xyz="0.0 0.0 ${forearm_length}" rpy="0.0 ${pi / 2.0} 0.0" /> -->
+      <!-- <origin xyz="0.0 0.0 ${forearm_length}" rpy="0.0 -2.09439 0.0" />  <!- do not know why ${-2.0 * pi / 3.0} collapses ODE --> -->
       <origin xyz="0.0 0.0 ${forearm_length}" rpy="0.0 ${pi / 3.0} 0.0" />
       <axis xyz="0 1 0" />
@@ -211,6 +204,6 @@
         </geometry>
       </collision>
-      <xacro:cylinder_inertial radius="0.6" length="0.12" mass="${wrist_1_mass}">
-        <origin xyz="0.0 0.0 0.0" rpy="0 0 0" />
+      <xacro:cylinder_inertial radius="0.06" length="0.12" mass="${wrist_1_mass}">
+        <origin xyz="0.0 ${wrist_1_length} 0.0" rpy="0 0 0" />
       </xacro:cylinder_inertial>
     </link>
@@ -242,6 +235,6 @@
         </geometry>
       </collision>
-      <xacro:cylinder_inertial radius="0.6" length="0.12" mass="${wrist_2_mass}">
-        <origin xyz="0.0 0.0 0.0" rpy="0 0 0" />
+      <xacro:cylinder_inertial radius="0.06" length="0.12" mass="${wrist_2_mass}">
+        <origin xyz="0.0 0.0 ${wrist_2_length}" rpy="0 0 0" />
       </xacro:cylinder_inertial>
     </link>
@@ -273,9 +266,9 @@
         </geometry>
       </collision>
-      <xacro:cylinder_inertial radius="0.6" length="0.12" mass="${wrist_3_mass}">
-        <origin xyz="0.0 0.0 0.0" rpy="0 0 0" />
-      </xacro:cylinder_inertial>
-    </link>
-    <joint name="${prefix}ee_fixed_joint_r" type="fixed">
+      <xacro:cylinder_inertial radius="0.0375" length="0.0345" mass="${wrist_3_mass}">
+        <origin xyz="0.0 ${wrist_3_length - 0.0345/2.0} 0.0" rpy="0 0 0" />
+      </xacro:cylinder_inertial>
+    </link>
+    <!-- <joint name="${prefix}ee_fixed_joint_r" type="fixed">
       <parent link="${prefix}wrist_3_link_r" />
       <child link = "${prefix}ee_link_r" />
@@ -289,25 +282,25 @@
         <origin rpy="0 0 0" xyz="-0.01 0 0"/>
       </collision>
-    </link>
+    </link> -->
     <xacro:ur_arm_transmission prefix="${prefix}" />
     <xacro:ur_arm_gazebo prefix="${prefix}" />
     <!-- ROS base_link to UR 'Base' Coordinates transform -->
-    <link name="${prefix}base_r"/>
-    <joint name="${prefix}base_link_r-base_fixed_joint" type="fixed">
+    <!-- <link name="${prefix}base_r"/>
+    <joint name="${prefix}base_link_r-base_fixed_joint" type="fixed"> -->
       <!-- NOTE: this rotation is only needed as long as base_link itself is
                  not corrected wrt the real robot (ie: rotated over 180
                  degrees)
       -->
-      <origin xyz="0 0 0" rpy="0 0 ${-pi}"/>
+      <!-- <origin xyz="0 0 0" rpy="0 0 ${-pi}"/>
       <parent link="${prefix}base_link_r"/>
       <child link="${prefix}base_r"/>
-    </joint>
+    </joint> -->
     <!-- Frame coincident with all-zeros TCP on UR controller -->
-    <link name="${prefix}tool0_r"/>
+    <!-- <link name="${prefix}tool0_r"/>
     <joint name="${prefix}wrist_3_link_r-tool0_fixed_joint" type="fixed">
       <origin xyz="0 ${wrist_3_length} 0" rpy="${pi/-2.0} 0 0"/>
       <parent link="${prefix}wrist_3_link_r"/>
       <child link="${prefix}tool0_r"/>
-    </joint>
+    </joint> -->
     <link name="${prefix}base_link_l" >
       <visual>
@@ -418,6 +411,6 @@
         </geometry>
       </collision>
-      <xacro:cylinder_inertial radius="0.06" length="0.5" mass="${forearm_mass}">
-        <origin xyz="0.0 0.0 0.25" rpy="0 0 0" />
+      <xacro:cylinder_inertial radius="0.06" length="${-ur5_a3}" mass="${forearm_mass}">
+        <origin xyz="0.0 0.0 ${-ur5_a3/2.0}" rpy="0 0 0" />
       </xacro:cylinder_inertial>
     </link>
@@ -425,5 +418,5 @@
       <parent link="${prefix}forearm_link_l" />
       <child link = "${prefix}wrist_1_link_l" />
-      <!-- <origin xyz="0.0 0.0 ${forearm_length}" rpy="0.0 ${pi / 2.0} 0.0" /> -->
+      <!-- <origin xyz="0.0 0.0 ${forearm_length}" rpy="0.0 2.09439 0.0" />  <! do not know why ${2.0 * pi / 3.0} collapses ODE --> -->
       <origin xyz="0.0 0.0 ${forearm_length}" rpy="0.0 ${-pi / 3.0} 0.0" />
       <axis xyz="0 1 0" />
@@ -450,6 +443,6 @@
         </geometry>
       </collision>
-      <xacro:cylinder_inertial radius="0.6" length="0.12" mass="${wrist_1_mass}">
-        <origin xyz="0.0 0.0 0.0" rpy="0 0 0" />
+      <xacro:cylinder_inertial radius="0.06" length="0.12" mass="${wrist_1_mass}">
+        <origin xyz="0.0 ${wrist_1_length} 0.0" rpy="0 0 0" />
       </xacro:cylinder_inertial>
     </link>
@@ -481,6 +474,6 @@
         </geometry>
       </collision>
-      <xacro:cylinder_inertial radius="0.6" length="0.12" mass="${wrist_2_mass}">
-        <origin xyz="0.0 0.0 0.0" rpy="0 0 0" />
+      <xacro:cylinder_inertial radius="0.06" length="0.12" mass="${wrist_2_mass}">
+        <origin xyz="0.0 0.0 ${wrist_2_length}" rpy="0 0 0" />
       </xacro:cylinder_inertial>
     </link>
@@ -512,14 +505,14 @@
         </geometry>
       </collision>
-      <xacro:cylinder_inertial radius="0.6" length="0.12" mass="${wrist_3_mass}">
-        <origin xyz="0.0 0.0 0.0" rpy="0 0 0" />
-      </xacro:cylinder_inertial>
-    </link>
-    <joint name="${prefix}ee_fixed_joint_l" type="fixed">
+      <xacro:cylinder_inertial radius="0.0375" length="0.0345" mass="${wrist_3_mass}">
+        <origin xyz="0.0 ${wrist_3_length - 0.0345/2} 0.0" rpy="0 0 0" />
+      </xacro:cylinder_inertial>
+    </link>
+    <!-- <joint name="${prefix}ee_fixed_joint_l" type="fixed">
       <parent link="${prefix}wrist_3_link_l" />
       <child link = "${prefix}ee_link_l" />
       <origin xyz="0.0 ${wrist_3_length} 0.0" rpy="0.0 0.0 ${pi/2.0}" />
-    </joint>
-    <link name="${prefix}ee_link_l">
+    </joint> -->
+    <!-- <link name="${prefix}ee_link_l">
       <collision>
         <geometry>
@@ -528,27 +521,31 @@
         <origin rpy="0 0 0" xyz="-0.01 0 0"/>
       </collision>
-    </link>
+    </link> -->
     <!-- ROS base_link to UR 'Base' Coordinates transform -->
-    <link name="${prefix}base_l"/>
+    <!-- <link name="${prefix}base_l"/>
     <joint name="${prefix}base_link_l-base_fixed_joint" type="fixed">
       <origin xyz="0 0 0" rpy="0 0 ${-pi}"/>
       <parent link="${prefix}base_link_l"/>
       <child link="${prefix}base_l"/>
-    </joint>
+    </joint> -->
     <!-- Frame coincident with all-zeros TCP on UR controller -->
-    <link name="${prefix}tool0_l"/>
+    <!-- <link name="${prefix}tool0_l"/>
     <joint name="${prefix}wrist_3_link_l-tool0_fixed_joint" type="fixed">
       <origin xyz="0 ${wrist_3_length} 0" rpy="${pi/-2.0} 0 0"/>
       <parent link="${prefix}wrist_3_link_l"/>
       <child link="${prefix}tool0_l"/>
-    </joint>
-    <joint name="wrist_3_to_obj_joint_r" type="fixed">
-        <origin rpy="0 0 0" xyz="0 ${wrist_3_length} 0"/>
-        <parent link="${prefix}wrist_3_link_r"/>
-        <child link="obj"/>
-    </joint>
-    <link name="obj">
+    </joint> -->
+    <!-- URDF parser eliminates 'fixed' joints: -->
+    <joint name="wrist_3_to_obj_joint_r" type="revolute">
+        <parent link="${prefix}wrist_3_link_r" />
+        <child link = "obj_link" />
+        <origin xyz="0.0 ${wrist_3_length} 0.0" rpy="0.0 0.0 0.0" />
+        <axis xyz="0 1 0" />
+        <limit lower="0.0" upper="0.0" effort="0.0" velocity="0.0"/>
+        <dynamics damping="0.0" friction="0.0"/>
+    </joint>
+    <link name="obj_link">
         <visual>
-            <origin rpy="0 0 0" xyz="0.0 ${obj_length/2} 0.0"/>
+            <origin rpy="0 0 0" xyz="0.0 ${obj_length/2.0} 0.0"/>
             <geometry>
                 <box size="0.05 ${obj_length} 0.05"/>
@@ -557,5 +554,5 @@
         </visual>
         <collision>
-            <origin rpy="0 0 0" xyz="0.0 ${obj_length/2} 0.0"/>
+            <origin rpy="0 0 0" xyz="0.0 ${obj_length/2.0} 0.0"/>
             <geometry>
                 <box size="0.05 ${obj_length} 0.05"/>
@@ -563,14 +560,14 @@
         </collision>
         <inertial>
-            <origin rpy="0 0 0" xyz="0.0 ${obj_length/2} 0.0"/>
+            <origin rpy="0 0 0" xyz="0.0 ${obj_length/2.0} 0.0"/>
             <mass value="${obj_mass}"/>
             <inertia ixx=".0021" ixy="0" ixz="0" iyy=".00021" iyz="0" izz=".0021"/>
         </inertial>
     </link>
-    <gazebo>
+    <!-- <gazebo>
         <joint name="wrist_3_to_obj_joint_l" type="fixed">
-            <parent>wrist_3_link_l</parent>
-            <child>obj</child>
-            <pose>0 ${obj_length + wrist_3_length} 0 0 0 0</pose>
+            <parent>${prefix}wrist_3_link_l</parent>
+            <child>obj_link</child>
+            <pose>0 ${obj_length} 0 0 0 0</pose>
             <physics>
                 <ode>
@@ -584,5 +581,56 @@
             </physics>
         </joint>
-    </gazebo>
+    </gazebo> -->
+    <!-- The ft_sensor plugin -->
+    <gazebo reference="wrist_3_to_obj_joint_r">
+        <provideFeedback>true</provideFeedback>
+    </gazebo>
+    <gazebo>
+        <plugin name="ft_sensor_obj_joint_r" filename="libgazebo_ros_ft_sensor.so">
+            <updateRate>100.0</updateRate>
+            <topicName>ft_sensor_topic_obj</topicName>
+            <jointName>wrist_3_to_obj_joint_r</jointName>
+        </plugin>
+    </gazebo>
+    <gazebo reference="${prefix}wrist_3_joint_r">
+        <provideFeedback>true</provideFeedback>
+    </gazebo>
+    <gazebo>
+        <plugin name="ft_sensor_wrist_r" filename="libgazebo_ros_ft_sensor.so">
+            <updateRate>100.0</updateRate>
+            <topicName>ft_sensor_topic_wrist_r</topicName>
+            <jointName>${prefix}wrist_3_joint_r</jointName>
+        </plugin>
+    </gazebo>
+    <!-- <gazebo reference="${prefix}wrist_3_joint_l">
+        <provideFeedback>true</provideFeedback>
+    </gazebo>
+    <gazebo>
+        <plugin name="ft_sensor_l" filename="libgazebo_ros_ft_sensor.so">
+            <updateRate>100.0</updateRate>
+            <topicName>ft_sensor_topic_l</topicName>
+            <jointName>${prefix}wrist_3_joint_l</jointName>
+        </plugin>
+    </gazebo> -->
+    <!-- <gazebo reference="wrist_3_to_obj_joint_r">
+        <provideFeedback>true</provideFeedback>
+    </gazebo>
+    <gazebo>
+        <plugin name="ft_sensor_r" filename="libgazebo_ros_ft_sensor.so">
+            <updateRate>100.0</updateRate>
+            <topicName>ft_sensor_topic_r</topicName>
+            <jointName>wrist_3_to_obj_joint_r</jointName>
+        </plugin>
+    </gazebo>
+    <gazebo reference="${prefix}wrist_3_joint_l">
+        <provideFeedback>true</provideFeedback>
+    </gazebo>
+    <gazebo>
+        <plugin name="ft_sensor_l" filename="libgazebo_ros_ft_sensor.so">
+            <updateRate>100.0</updateRate>
+            <topicName>ft_sensor_topic_l</topicName>
+            <jointName>${prefix}wrist_3_joint_l</jointName>
+        </plugin>
+    </gazebo> -->
   </xacro:macro>
 </robot>

File: ur5_description/urdf/ur5_left_joint_limited_robot.urdf (robot description, URDF)
Before this commit: robot ur5, 11 links, 10 joints
Links:
- removed link base_l
- removed link ee_link_l
- removed link tool0_l
Joints:
- removed joint base_link_l-base_fixed_joint
- removed joint ee_fixed_joint_l
- removed joint wrist_3_link_l-tool0_fixed_joint

File: ur5_description/urdf/ur5_right_joint_limited_robot.urdf (robot description, URDF)
Before this commit: robot ur5, 11 links, 10 joints
Links:
- removed link base_r
- removed link ee_link_r
- removed link tool0_r
Joints:
- removed joint base_link_r-base_fixed_joint
- removed joint ee_fixed_joint_r
- removed joint wrist_3_link_r-tool0_fixed_joint

Commit message: `wrist_3_joint_r` FT sensor added to compare with `lambda_r`.

File: ur5_description/urdf/ur5.urdf.xacro (robot description, xacro)
@@ -548,4 +548,17 @@
         <child link="obj"/>
     </joint>
+    <!-- <joint name="${prefix}wrist3_obj_joint_r" type="revolute">
+      <parent link="${prefix}wrist_3_link_r" />
+      <child link = "obj" />
+      <origin rpy="0 0 0" xyz="0 ${wrist_3_length} 0"/>
+      <axis xyz="0 1 0" />
+      <xacro:unless value="${joint_limited}">
+        <limit lower="0." upper="0." effort="0." velocity="0."/>
+      </xacro:unless>
+      <xacro:if value="${joint_limited}">
+        <limit lower="0." upper="0." effort="0." velocity="0."/>
+      </xacro:if>
+      <dynamics damping="0.0" friction="0.0"/>
+    </joint> -->
     <link name="obj">
         <visual>
@@ -585,4 +598,14 @@
         </joint>
     </gazebo>
+    <gazebo reference="${prefix}wrist_3_joint_r">
+        <provideFeedback>true</provideFeedback>
+    </gazebo>
+    <gazebo>
+        <plugin name="ft_sensor_wrist3_r" filename="libgazebo_ros_ft_sensor.so">
+            <updateRate>100.0</updateRate>
+            <topicName>ft_sensor_topic_wrist3_r</topicName>
+            <jointName>${prefix}wrist_3_joint_r</jointName>
+        </plugin>
+    </gazebo>
   </xacro:macro>
 </robot>
